File: hardware/esp-mhi-ac.kicad_sch (KiCad schematic)
At the start: 15 parts, among them J1 CNS AC, J2 LS-HV, J3 LS-LV, J4 ADA BMEx80, J5 BMEx80, J6 BH1750, U1 WeMos_D1_mini, U2 TSR_1-2450

Commit message: update hardware
Parts:
- added JP1: BME680 ADDR, Jumper:SolderJumper-2_P1.3mm_Open_TrianglePad1.0x1.5mm, symbol Jumper:SolderJumper_2_Open
- added JP2: BH1750 ADDR, Jumper:SolderJumper-2_P1.3mm_Open_TrianglePad1.0x1.5mm, symbol Jumper:SolderJumper_2_Open
- J1: footprint Connector_JST:JST_XH_B5B-XH-A_1x05_P2.50mm_Vertical -> Connector_JST:JST_XH_S5B-XH-A_1x05_P2.50mm_Horizontal
Connections:
- net +3.3V: now also JP2.1 (A)
- net GND: now also JP1.1 (A)
- net at J4.3 (Pin_3): now also JP1.2 (B)
- net at J6.1 (Pin_1): now also JP2.2 (B)
- no-connect marks 16 -> 14
Other:
- moved on the sheet: J4
Changed lines of the file:
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@@
   (junction (at 63.5 40.64) (diameter 0) (color 0 0 0 0)
   )
+  (junction (at 106.68 40.64) (diameter 0) (color 0 0 0 0)
+  )
   (junction (at 41.91 31.75) (diameter 0) (color 0 0 0 0)
+  )
+  (junction (at 120.65 77.47) (diameter 0) (color 0 0 0 0)
   )
   (junction (at 54.61 40.64) (diameter 0) (color 0 0 0 0)
@@
   (no_connect (at 48.26 96.52))
   (no_connect (at 48.26 83.82))
+  (no_connect (at 124.46 38.1))
   (no_connect (at 48.26 86.36))
   (no_connect (at 106.68 90.17))
@@
   (no_connect (at 71.12 66.04))
   (no_connect (at 81.28 90.17))
-  (no_connect (at 96.52 68.58))
   (no_connect (at 27.94 76.2))
   (no_connect (at 27.94 83.82))
-  (no_connect (at 133.35 67.31))
   (no_connect (at 48.26 76.2))
   (no_connect (at 48.26 73.66))
-  (no_connect (at 96.52 76.2))
   (no_connect (at 71.12 68.58))
-  (no_connect (at 96.52 63.5))
+  (no_connect (at 124.46 25.4))
+  (wire (pts (xy 106.68 30.48) (xy 124.46 30.48))
+    (stroke (width 0) (type default))
+  )
   (wire (pts (xy 30.48 39.37) (xy 30.48 40.64))
     (stroke (width 0) (type default))
@@
     (stroke (width 0) (type default))
   )
+  (wire (pts (xy 111.76 40.64) (xy 106.68 40.64))
+    (stroke (width 0) (type default))
+  )
   (wire (pts (xy 35.56 64.77) (xy 35.56 66.04))
     (stroke (width 0) (type default))
@@
     (stroke (width 0) (type default))
   )
+  (wire (pts (xy 120.65 74.93) (xy 120.65 77.47))
+    (stroke (width 0) (type default))
+  )
   (wire (pts (xy 106.68 95.25) (xy 113.03 95.25))
     (stroke (width 0) (type default))
@@
     (stroke (width 0) (type default))
   )
+  (wire (pts (xy 120.65 67.31) (xy 133.35 67.31))
+    (stroke (width 0) (type default))
+  )
+  (wire (pts (xy 120.65 77.47) (xy 133.35 77.47))
+    (stroke (width 0) (type default))
+  )
+  (wire (pts (xy 106.68 30.48) (xy 106.68 33.02))
+    (stroke (width 0) (type default))
+  )
   (wire (pts (xy 40.64 62.23) (xy 40.64 66.04))
     (stroke (width 0) (type default))
@@
     (stroke (width 0) (type default))
   )
+  (wire (pts (xy 124.46 35.56) (xy 111.76 35.56))
+    (stroke (width 0) (type default))
+  )
   (wire (pts (xy 41.91 31.75) (xy 53.34 31.75))
+    (stroke (width 0) (type default))
+  )
+  (wire (pts (xy 111.76 35.56) (xy 111.76 40.64))
     (stroke (width 0) (type default))
   )
@@
     )
   )
-  (global_label "SCL" (shape input) (at 96.52 71.12 180) (fields_autoplaced)
+  (global_label "SCL" (shape input) (at 124.46 33.02 180) (fields_autoplaced)
     (effects (font (size 1.27 1.27)) (justify right))
-    (property "Intersheetrefs" "${INTERSHEET_REFS}" (at 90.0272 71.12 0)
+    (property "Intersheetrefs" "${INTERSHEET_REFS}" (at 117.9672 33.02 0)
       (effects (font (size 1.27 1.27)) (justify right) hide)
     )
@@
     )
   )
-  (global_label "SDA" (shape input) (at 96.52 66.04 180) (fields_autoplaced)
+  (global_label "SDA" (shape input) (at 124.46 27.94 180) (fields_autoplaced)
     (effects (font (size 1.27 1.27)) (justify right))
-    (property "Intersheetrefs" "${INTERSHEET_REFS}" (at 89.9667 66.04 0)
+    (property "Intersheetrefs" "${INTERSHEET_REFS}" (at 117.9067 27.94 0)
       (effects (font (size 1.27 1.27)) (justify right) hide)
     )
@@
     )
   )
-  (symbol (lib_id "power:+3.3V") (at 96.52 78.74 90) (unit 1)
-    (in_bom yes) (on_board yes) (dnp no) (fields_autoplaced)
-    (property "Reference" "#PWR013" (at 100.33 78.74 0)
-      (effects (font (size 1.27 1.27)) hide)
-    )
-    (property "Value" "+3.3V" (at 92.71 78.74 90)
-      (effects (font (size 1.27 1.27)) (justify left))
-    )
-    (property "Footprint" "" (at 96.52 78.74 0)
-      (effects (font (size 1.27 1.27)) hide)
-    )
-    (property "Datasheet" "" (at 96.52 78.74 0)
+  (symbol (lib_id "power:+3.3V") (at 124.46 40.64 90) (unit 1)
+    (in_bom yes) (on_board yes) (dnp no) (fields_autoplaced)
+    (property "Reference" "#PWR013" (at 128.27 40.64 0)
+      (effects (font (size 1.27 1.27)) hide)
+    )
+    (property "Value" "+3.3V" (at 120.65 40.64 90)
+      (effects (font (size 1.27 1.27)) (justify left))
+    )
+    (property "Footprint" "" (at 124.46 40.64 0)
+      (effects (font (size 1.27 1.27)) hide)
+    )
+    (property "Datasheet" "" (at 124.46 40.64 0)
       (effects (font (size 1.27 1.27)) hide)
     )
@@
     )
   )
-  (symbol (lib_id "Connector_Generic:Conn_01x07") (at 101.6 71.12 0) (unit 1)
-    (in_bom yes) (on_board yes) (dnp no) (fields_autoplaced)
-    (property "Reference" "J4" (at 104.14 69.85 0)
-      (effects (font (size 1.27 1.27)) (justify left))
-    )
-    (property "Value" "ADA BMEx80" (at 104.14 72.39 0)
-      (effects (font (size 1.27 1.27)) (justify left))
-    )
-    (property "Footprint" "Connector_PinSocket_2.54mm:PinSocket_1x07_P2.54mm_Vertical" (at 101.6 71.12 0)
-      (effects (font (size 1.27 1.27)) hide)
-    )
-    (property "Datasheet" "~" (at 101.6 71.12 0)
+  (symbol (lib_id "Jumper:SolderJumper_2_Open") (at 120.65 71.12 90) (unit 1)
+    (in_bom yes) (on_board yes) (dnp no)
+    (property "Reference" "JP2" (at 115.57 69.85 90)
+      (effects (font (size 1.27 1.27)) (justify right))
+    )
+    (property "Value" "BH1750 ADDR" (at 105.41 73.66 90)
+      (effects (font (size 1.27 1.27)) (justify right))
+    )
+    (property "Footprint" "Jumper:SolderJumper-2_P1.3mm_Open_TrianglePad1.0x1.5mm" (at 120.65 71.12 0)
+      (effects (font (size 1.27 1.27)) hide)
+    )
+    (property "Datasheet" "~" (at 120.65 71.12 0)
+      (effects (font (size 1.27 1.27)) hide)
+    )
+    (pin "1")
+    (pin "2")
+    (instances
+      (project "esp-mhi-ac"
+        (path "/8e1a3eac-db9c-4223-ad01-db8aab4e8a86"
+          (reference "JP2") (unit 1)
+        )
+      )
+    )
+  )
+  (symbol (lib_id "Connector_Generic:Conn_01x07") (at 129.54 33.02 0) (unit 1)
+    (in_bom yes) (on_board yes) (dnp no) (fields_autoplaced)
+    (property "Reference" "J4" (at 132.08 31.75 0)
+      (effects (font (size 1.27 1.27)) (justify left))
+    )
+    (property "Value" "ADA BMEx80" (at 132.08 34.29 0)
+      (effects (font (size 1.27 1.27)) (justify left))
+    )
+    (property "Footprint" "Connector_PinSocket_2.54mm:PinSocket_1x07_P2.54mm_Vertical" (at 129.54 33.02 0)
+      (effects (font (size 1.27 1.27)) hide)
+    )
+    (property "Datasheet" "~" (at 129.54 33.02 0)
       (effects (font (size 1.27 1.27)) hide)
     )
@@
     )
   )
-  (symbol (lib_id "power:+3.3V") (at 133.35 77.47 90) (unit 1)
-    (in_bom yes) (on_board yes) (dnp no) (fields_autoplaced)
-    (property "Reference" "#PWR07" (at 137.16 77.47 0)
-      (effects (font (size 1.27 1.27)) hide)
-    )
-    (property "Value" "+3.3V" (at 129.54 77.47 90)
-      (effects (font (size 1.27 1.27)) (justify left))
-    )
-    (property "Footprint" "" (at 133.35 77.47 0)
-      (effects (font (size 1.27 1.27)) hide)
-    )
-    (property "Datasheet" "" (at 133.35 77.47 0)
+  (symbol (lib_id "power:+3.3V") (at 120.65 77.47 180) (unit 1)
+    (in_bom yes) (on_board yes) (dnp no) (fields_autoplaced)
+    (property "Reference" "#PWR07" (at 120.65 73.66 0)
+      (effects (font (size 1.27 1.27)) hide)
+    )
+    (property "Value" "+3.3V" (at 120.65 82.55 0)
+      (effects (font (size 1.27 1.27)))
+    )
+    (property "Footprint" "" (at 120.65 77.47 0)
+      (effects (font (size 1.27 1.27)) hide)
+    )
+    (property "Datasheet" "" (at 120.65 77.47 0)
       (effects (font (size 1.27 1.27)) hide)
     )
@@
     )
   )
+  (symbol (lib_id "Jumper:SolderJumper_2_Open") (at 106.68 36.83 90) (unit 1)
+    (in_bom yes) (on_board yes) (dnp no)
+    (property "Reference" "JP1" (at 101.6 35.56 90)
+      (effects (font (size 1.27 1.27)) (justify right))
+    )
+    (property "Value" "BME680 ADDR" (at 91.44 39.37 90)
+      (effects (font (size 1.27 1.27)) (justify right))
+    )
+    (property "Footprint" "Jumper:SolderJumper-2_P1.3mm_Open_TrianglePad1.0x1.5mm" (at 106.68 36.83 0)
+      (effects (font (size 1.27 1.27)) hide)
+    )
+    (property "Datasheet" "~" (at 106.68 36.83 0)
+      (effects (font (size 1.27 1.27)) hide)
+    )
+    (pin "1")
+    (pin "2")
+    (instances
+      (project "esp-mhi-ac"
+        (path "/8e1a3eac-db9c-4223-ad01-db8aab4e8a86"
+          (reference "JP1") (unit 1)
+        )
+      )
+    )
+  )
   (symbol (lib_id "power:GND") (at 71.12 76.2 270) (unit 1)
     (in_bom yes) (on_board yes) (dnp no) (fields_autoplaced)
@@
     )
   )
-  (symbol (lib_id "power:GND") (at 96.52 73.66 270) (unit 1)
-    (in_bom yes) (on_board yes) (dnp no) (fields_autoplaced)
-    (property "Reference" "#PWR012" (at 90.17 73.66 0)
-      (effects (font (size 1.27 1.27)) hide)
-    )
-    (property "Value" "GND" (at 92.71 73.66 90)
-      (effects (font (size 1.27 1.27)) (justify right))
-    )
-    (property "Footprint" "" (at 96.52 73.66 0)
-      (effects (font (size 1.27 1.27)) hide)
-    )
-    (property "Datasheet" "" (at 96.52 73.66 0)
+  (symbol (lib_id "power:GND") (at 106.68 40.64 0) (unit 1)
+    (in_bom yes) (on_board yes) (dnp no) (fields_autoplaced)
+    (property "Reference" "#PWR012" (at 106.68 46.99 0)
+      (effects (font (size 1.27 1.27)) hide)
+    )
+    (property "Value" "GND" (at 109.22 41.91 0)
+      (effects (font (size 1.27 1.27)) (justify left))
+    )
+    (property "Footprint" "" (at 106.68 40.64 0)
+      (effects (font (size 1.27 1.27)) hide)
+    )
+    (property "Datasheet" "" (at 106.68 40.64 0)
       (effects (font (size 1.27 1.27)) hide)
     )
@@
       (effects (font (size 1.27 1.27)) (justify left))
     )
-    (property "Footprint" "Connector_JST:JST_XH_B5B-XH-A_1x05_P2.50mm_Vertical" (at 138.43 96.52 0)
-      (effects (font (size 1.27 1.27)) hide)
-    )
+    (property "Footprint" "Connector_JST:JST_XH_S5B-XH-A_1x05_P2.50mm_Horizontal" (at 138.43 96.52 0)
+      (effects (font (size 1.27 1.27)) hide)
+    )
